File: Kicad/board.kicad_sch (KiCad schematic)
At the start: 45 parts, among them SW1 SW_Push, SW10 SW_Push, SW11 SW_Push, SW12 SW_Push, SW13 RotaryEncoder, SW2 SW_Push, SW3 SW_Push, SW4 SW_Push, SW5 SW_Push, SW6 SW_Push, SW7 SW_Push, SW8 SW_Push, SW9 SW_Push, U1 XIAO-ESP32-S3-DIP, U2 KY-023, U3 OLED, U4 KY-023

Commit message: [update] update diode footprint
Parts:
- D1, D10, D11, D12, D2, D3, D4, D5, D6, D7, D8, D9: value 1N4148W -> 1N4148; footprint Diode_THT:D_DO-35_SOD27_P7.62mm_Horizontal -> mylib:Diode_THT_reversible
- SW1, SW10, SW11, SW12, SW2, SW3, SW4, SW5, SW6, SW7, SW8, SW9: footprint keyswitches:Kailh_socket_PG1350_optional_reversible -> mylib:Kailh_socket_PG1350_optional_reversible
- U3: footprint (none) -> Connector_PinSocket_2.54mm:PinSocket_1x05_P2.54mm_Vertical
Changed lines of the file:
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@@
 			)
 		)
-		(property "Value" "1N4148W"
+		(property "Value" "1N4148"
 			(at 110.49 55.8799 90)
 			(effects
@@
 			)
 		)
-		(property "Footprint" "Diode_THT:D_DO-35_SOD27_P7.62mm_Horizontal"
+		(property "Footprint" "mylib:Diode_THT_reversible"
 			(at 112.395 54.61 0)
 			(effects
@@
 			)
 		)
-		(property "Footprint" "keyswitches:Kailh_socket_PG1350_optional_reversible"
+		(property "Footprint" "mylib:Kailh_socket_PG1350_optional_reversible"
 			(at 102.87 71.12 0)
 			(effects
@@
 			)
 		)
-		(property "Footprint" "keyswitches:Kailh_socket_PG1350_optional_reversible"
+		(property "Footprint" "mylib:Kailh_socket_PG1350_optional_reversible"
 			(at 77.47 71.12 0)
 			(effects
@@
 			)
 		)
-		(property "Value" "1N4148W"
+		(property "Value" "1N4148"
 			(at 135.89 55.8799 90)
 			(effects
@@
 			)
 		)
-		(property "Footprint" "Diode_THT:D_DO-35_SOD27_P7.62mm_Horizontal"
+		(property "Footprint" "mylib:Diode_THT_reversible"
 			(at 137.795 54.61 0)
 			(effects
@@
 			)
 		)
-		(property "Footprint" ""
+		(property "Footprint" "Connector_PinSocket_2.54mm:PinSocket_1x05_P2.54mm_Vertical"
 			(at 123.19 123.19 0)
 			(effects
@@
 			)
 		)
-		(property "Value" "1N4148W"
+		(property "Value" "1N4148"
 			(at 135.89 81.2799 90)
 			(effects
@@
 			)
 		)
-		(property "Footprint" "Diode_THT:D_DO-35_SOD27_P7.62mm_Horizontal"
+		(property "Footprint" "mylib:Diode_THT_reversible"
 			(at 137.795 80.01 0)
 			(effects
@@
 			)
 		)
-		(property "Footprint" "keyswitches:Kailh_socket_PG1350_optional_reversible"
+		(property "Footprint" "mylib:Kailh_socket_PG1350_optional_reversible"
 			(at 102.87 58.42 0)
 			(effects
@@
 			)
 		)
-		(property "Footprint" "keyswitches:Kailh_socket_PG1350_optional_reversible"
+		(property "Footprint" "mylib:Kailh_socket_PG1350_optional_reversible"
 			(at 128.27 58.42 0)
 			(effects
@@
 			)
 		)
-		(property "Value" "1N4148W"
+		(property "Value" "1N4148"
 			(at 85.09 68.5799 90)
 			(effects
@@
 			)
 		)
-		(property "Footprint" "Diode_THT:D_DO-35_SOD27_P7.62mm_Horizontal"
+		(property "Footprint" "mylib:Diode_THT_reversible"
 			(at 86.995 67.31 0)
 			(effects
@@
 			)
 		)
-		(property "Value" "1N4148W"
+		(property "Value" "1N4148"
 			(at 59.69 81.2799 90)
 			(effects
@@
 			)
 		)
-		(property "Footprint" "Diode_THT:D_DO-35_SOD27_P7.62mm_Horizontal"
+		(property "Footprint" "mylib:Diode_THT_reversible"
 			(at 61.595 80.01 0)
 			(effects
@@
 			)
 		)
-		(property "Value" "1N4148W"
+		(property "Value" "1N4148"
 			(at 85.09 81.2799 90)
 			(effects
@@
 			)
 		)
-		(property "Footprint" "Diode_THT:D_DO-35_SOD27_P7.62mm_Horizontal"
+		(property "Footprint" "mylib:Diode_THT_reversible"
 			(at 86.995 80.01 0)
 			(effects
@@
 			)
 		)
-		(property "Footprint" "keyswitches:Kailh_socket_PG1350_optional_reversible"
+		(property "Footprint" "mylib:Kailh_socket_PG1350_optional_reversible"
 			(at 128.27 71.12 0)
 			(effects
@@
 			)
 		)
-		(property "Value" "1N4148W"
+		(property "Value" "1N4148"
 			(at 135.89 68.5799 90)
 			(effects
@@
 			)
 		)
-		(property "Footprint" "Diode_THT:D_DO-35_SOD27_P7.62mm_Horizontal"
+		(property "Footprint" "mylib:Diode_THT_reversible"
 			(at 137.795 67.31 0)
 			(effects
@@
 			)
 		)
-		(property "Footprint" "keyswitches:Kailh_socket_PG1350_optional_reversible"
+		(property "Footprint" "mylib:Kailh_socket_PG1350_optional_reversible"
 			(at 128.27 45.72 0)
 			(effects
@@
 			)
 		)
-		(property "Footprint" "keyswitches:Kailh_socket_PG1350_optional_reversible"
+		(property "Footprint" "mylib:Kailh_socket_PG1350_optional_reversible"
 			(at 52.07 58.42 0)
 			(effects
@@
 			)
 		)
-		(property "Value" "1N4148W"
+		(property "Value" "1N4148"
 			(at 110.49 81.2799 90)
 			(effects
@@
 			)
 		)
-		(property "Footprint" "Diode_THT:D_DO-35_SOD27_P7.62mm_Horizontal"
+		(property "Footprint" "mylib:Diode_THT_reversible"
 			(at 112.395 80.01 0)
 			(effects
@@
 			)
 		)
-		(property "Footprint" "keyswitches:Kailh_socket_PG1350_optional_reversible"
+		(property "Footprint" "mylib:Kailh_socket_PG1350_optional_reversible"
 			(at 52.07 45.72 0)
 			(effects
@@
 			)
 		)
-		(property "Footprint" "keyswitches:Kailh_socket_PG1350_optional_reversible"
+		(property "Footprint" "mylib:Kailh_socket_PG1350_optional_reversible"
 			(at 102.87 45.72 0)
 			(effects
@@
 			)
 		)
-		(property "Value" "1N4148W"
+		(property "Value" "1N4148"
 			(at 59.69 68.5799 90)
 			(effects
@@
 			)
 		)
-		(property "Footprint" "Diode_THT:D_DO-35_SOD27_P7.62mm_Horizontal"
+		(property "Footprint" "mylib:Diode_THT_reversible"
 			(at 61.595 67.31 0)
 			(effects
@@
 			)
 		)
-		(property "Value" "1N4148W"
+		(property "Value" "1N4148"
 			(at 85.09 55.8799 90)
 			(effects
@@
 			)
 		)
-		(property "Footprint" "Diode_THT:D_DO-35_SOD27_P7.62mm_Horizontal"
+		(property "Footprint" "mylib:Diode_THT_reversible"
 			(at 86.995 54.61 0)
 			(effects
@@
 			)
 		)
-		(property "Value" "1N4148W"
+		(property "Value" "1N4148"
 			(at 110.49 68.5799 90)
 			(effects
@@
 			)
 		)
-		(property "Footprint" "Diode_THT:D_DO-35_SOD27_P7.62mm_Horizontal"
+		(property "Footprint" "mylib:Diode_THT_reversible"
 			(at 112.395 67.31 0)
 			(effects
@@
 			)
 		)
-		(property "Footprint" "keyswitches:Kailh_socket_PG1350_optional_reversible"
+		(property "Footprint" "mylib:Kailh_socket_PG1350_optional_reversible"
 			(at 52.07 71.12 0)
 			(effects
@@
 			)
 		)
-		(property "Value" "1N4148W"
+		(property "Value" "1N4148"
 			(at 59.69 55.8799 90)
 			(effects
@@
 			)
 		)
-		(property "Footprint" "Diode_THT:D_DO-35_SOD27_P7.62mm_Horizontal"
+		(property "Footprint" "mylib:Diode_THT_reversible"
 			(at 61.595 54.61 0)
 			(effects
@@
 			)
 		)
-		(property "Footprint" "keyswitches:Kailh_socket_PG1350_optional_reversible"
+		(property "Footprint" "mylib:Kailh_socket_PG1350_optional_reversible"
 			(at 77.47 45.72 0)
 			(effects
@@
 			)
 		)
-		(property "Footprint" "keyswitches:Kailh_socket_PG1350_optional_reversible"
+		(property "Footprint" "mylib:Kailh_socket_PG1350_optional_reversible"
 			(at 77.47 58.42 0)
 			(effects

Commit message: [update] re-annotate symbols
Parts:
- renumbered JP5 to JP1, JP6 to JP2, JP7 to JP3, JP8 to JP4, JP9 to JP5, JP10 to JP6, JP11 to JP7, JP12 to JP8
Changed lines of the file:
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@@
 		(on_board yes)
 		(dnp no)
-		(property "Reference" "JP5"
+		(property "Reference" "JP1"
 			(at 146.05 115.824 0)
 			(effects
@@
 			(project "board"
 				(path "/e49ea350-db18-4e55-8e96-c45c407ec11d"
-					(reference "JP5")
+					(reference "JP1")
 					(unit 1)
 				)
@@
 		(on_board yes)
 		(dnp no)
-		(property "Reference" "JP10"
+		(property "Reference" "JP6"
 			(at 146.05 145.034 0)
 			(effects
@@
 			(project "board"
 				(path "/e49ea350-db18-4e55-8e96-c45c407ec11d"
-					(reference "JP10")
+					(reference "JP6")
 					(unit 1)
 				)
@@
 		(dnp no)
 		(fields_autoplaced yes)
-		(property "Reference" "#PWR015"
+		(property "Reference" "#PWR09"
 			(at 149.86 123.19 0)
 			(effects
@@
 			(project "board"
 				(path "/e49ea350-db18-4e55-8e96-c45c407ec11d"
-					(reference "#PWR015")
+					(reference "#PWR09")
 					(unit 1)
 				)
@@
 		(dnp no)
 		(fields_autoplaced yes)
-		(property "Reference" "#PWR013"
+		(property "Reference" "#PWR016"
 			(at 219.71 154.94 0)
 			(effects
@@
 			(project "board"
 				(path "/e49ea350-db18-4e55-8e96-c45c407ec11d"
-					(reference "#PWR013")
+					(reference "#PWR016")
 					(unit 1)
 				)
@@
 		(dnp no)
 		(fields_autoplaced yes)
-		(property "Reference" "#PWR07"
+		(property "Reference" "#PWR05"
 			(at 133.35 118.11 0)
 			(effects
@@
 			(project "board"
 				(path "/e49ea350-db18-4e55-8e96-c45c407ec11d"
-					(reference "#PWR07")
+					(reference "#PWR05")
 					(unit 1)
 				)
@@
 		(dnp no)
 		(fields_autoplaced yes)
-		(property "Reference" "#PWR012"
+		(property "Reference" "#PWR014"
 			(at 219.71 149.86 0)
 			(effects
@@
 			(project "board"
 				(path "/e49ea350-db18-4e55-8e96-c45c407ec11d"
-					(reference "#PWR012")
+					(reference "#PWR014")
 					(unit 1)
 				)
@@
 		(on_board yes)
 		(dnp no)
-		(property "Reference" "JP6"
+		(property "Reference" "JP2"
 			(at 146.05 120.904 0)
 			(effects
@@
 			(project "board"
 				(path "/e49ea350-db18-4e55-8e96-c45c407ec11d"
-					(reference "JP6")
+					(reference "JP2")
 					(unit 1)
 				)
@@
 		(on_board yes)
 		(dnp no)
-		(property "Reference" "JP9"
+		(property "Reference" "JP5"
 			(at 146.05 139.954 0)
 			(effects
@@
 			(project "board"
 				(path "/e49ea350-db18-4e55-8e96-c45c407ec11d"
-					(reference "JP9")
+					(reference "JP5")
 					(unit 1)
 				)
@@
 		(on_board yes)
 		(dnp no)
-		(property "Reference" "JP8"
+		(property "Reference" "JP4"
 			(at 146.05 132.334 0)
 			(effects
@@
 			(project "board"
 				(path "/e49ea350-db18-4e55-8e96-c45c407ec11d"
-					(reference "JP8")
+					(reference "JP4")
 					(unit 1)
 				)
@@
 		(dnp no)
 		(fields_autoplaced yes)
-		(property "Reference" "#PWR06"
+		(property "Reference" "#PWR08"
 			(at 219.71 124.46 0)
 			(effects
@@
 			(project ""
 				(path "/e49ea350-db18-4e55-8e96-c45c407ec11d"
-					(reference "#PWR06")
+					(reference "#PWR08")
 					(unit 1)
 				)
@@
 		(dnp no)
 		(fields_autoplaced yes)
-		(property "Reference" "#PWR014"
+		(property "Reference" "#PWR013"
 			(at 160.02 142.24 0)
 			(effects
@@
 			(project "board"
 				(path "/e49ea350-db18-4e55-8e96-c45c407ec11d"
-					(reference "#PWR014")
+					(reference "#PWR013")
 					(unit 1)
 				)
@@
 		(on_board yes)
 		(dnp no)
-		(property "Reference" "JP12"
+		(property "Reference" "JP8"
 			(at 146.05 156.464 0)
 			(effects
@@
 			(project "board"
 				(path "/e49ea350-db18-4e55-8e96-c45c407ec11d"
-					(reference "JP12")
+					(reference "JP8")
 					(unit 1)
 				)
@@
 		(dnp no)
 		(fields_autoplaced yes)
-		(property "Reference" "#PWR016"
+		(property "Reference" "#PWR015"
 			(at 149.86 147.32 0)
 			(effects
@@
 			(project "board"
 				(path "/e49ea350-db18-4e55-8e96-c45c407ec11d"
-					(reference "#PWR016")
+					(reference "#PWR015")
 					(unit 1)
 				)
@@
 		(dnp no)
 		(fields_autoplaced yes)
-		(property "Reference" "#PWR010"
+		(property "Reference" "#PWR011"
 			(at 67.31 146.05 0)
 			(effects
@@
 			(project "board"
 				(path "/e49ea350-db18-4e55-8e96-c45c407ec11d"
-					(reference "#PWR010")
+					(reference "#PWR011")
 					(unit 1)
 				)
@@
 		(on_board yes)
 		(dnp no)
-		(property "Reference" "JP7"
+		(property "Reference" "JP3"
 			(at 146.05 125.984 0)
 			(effects
@@
 			(project "board"
 				(path "/e49ea350-db18-4e55-8e96-c45c407ec11d"
-					(reference "JP7")
+					(reference "JP3")
 					(unit 1)
 				)
@@
 		(dnp no)
 		(fields_autoplaced yes)
-		(property "Reference" "#PWR011"
+		(property "Reference" "#PWR012"
 			(at 78.74 146.05 0)
 			(effects
@@
 			(project ""
 				(path "/e49ea350-db18-4e55-8e96-c45c407ec11d"
-					(reference "#PWR011")
+					(reference "#PWR012")
 					(unit 1)
 				)
@@
 		(dnp no)
 		(fields_autoplaced yes)
-		(property "Reference" "#PWR05"
+		(property "Reference" "#PWR06"
 			(at 219.71 119.38 0)
 			(effects
@@
 			(project ""
 				(path "/e49ea350-db18-4e55-8e96-c45c407ec11d"
-					(reference "#PWR05")
+					(reference "#PWR06")
 					(unit 1)
 				)
@@
 		(on_board yes)
 		(dnp no)
-		(property "Reference" "JP11"
+		(property "Reference" "JP7"
 			(at 146.05 150.114 0)
 			(effects
@@
 			(project "board"
 				(path "/e49ea350-db18-4e55-8e96-c45c407ec11d"
-					(reference "JP11")
+					(reference "JP7")
 					(unit 1)
 				)
@@
 		(dnp no)
 		(fields_autoplaced yes)
-		(property "Reference" "#PWR08"
+		(property "Reference" "#PWR07"
 			(at 160.02 118.11 0)
 			(effects
@@
 			(project "board"
 				(path "/e49ea350-db18-4e55-8e96-c45c407ec11d"
-					(reference "#PWR08")
+					(reference "#PWR07")
 					(unit 1)
 				)
@@
 		(dnp no)
 		(fields_autoplaced yes)
-		(property "Reference" "#PWR09"
+		(property "Reference" "#PWR010"
 			(at 41.91 146.05 0)
 			(effects
@@
 			(project "board"
 				(path "/e49ea350-db18-4e55-8e96-c45c407ec11d"
-					(reference "#PWR09")
+					(reference "#PWR010")
 					(unit 1)
 				)

Commit message: [update] clear the ERC
Parts:
- C1, C2: footprint Capacitor_SMD:C_0805_2012Metric_Pad1.18x1.45mm_HandSolder -> mylib:C_0805_2012_HandSolder_reversible
- R1, R2: footprint Resistor_THT:R_Axial_DIN0207_L6.3mm_D2.5mm_P10.16mm_Horizontal -> mylib:R_L6.3mm_D2.5mm_P10.16mm_Horizontal_reversible
Connections:
- net VCC: now also U1.14 (VBUS); no longer U1.12 (VCC_3V3)
Changed lines of the file:
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@@
 	)
 	(junction
+		(at 246.38 57.15)
+		(diameter 0)
+		(color 0 0 0 0)
+	)
+	(junction
 		(at 41.91 124.46)
 		(diameter 0)
@@
 	)
 	(junction
+		(at 260.35 60.96)
+		(diameter 0)
+		(color 0 0 0 0)
+	)
+	(junction
 		(at 57.15 83.82)
 		(diameter 0)
@@
 	)
 	(no_connect
-		(at 243.84 57.15)
-	)
-	(no_connect
 		(at 46.99 88.9)
 	)
@@
 	)
 	(no_connect
+		(at 243.84 64.77)
+	)
+	(no_connect
 		(at 137.16 83.82)
 	)
@@
 	(wire
 		(pts
+			(xy 246.38 57.15) (xy 254 57.15)
+		)
+		(stroke
+			(width 0)
+			(type default)
+		)
+	)
+	(wire
+		(pts
 			(xy 107.95 71.12) (xy 133.35 71.12)
 		)
@@
 	(wire
 		(pts
-			(xy 67.31 121.92) (xy 67.31 129.54)
+			(xy 246.38 57.15) (xy 243.84 57.15)
 		)
 		(stroke
@@
 	(wire
 		(pts
-			(xy 78.74 127) (xy 78.74 140.97)
+			(xy 67.31 121.92) (xy 67.31 129.54)
 		)
 		(stroke
@@
 	(wire
 		(pts
-			(xy 107.95 83.82) (xy 133.35 83.82)
+			(xy 78.74 127) (xy 78.74 140.97)
 		)
 		(stroke
@@
 	(wire
 		(pts
-			(xy 243.84 64.77) (xy 248.92 64.77)
+			(xy 107.95 83.82) (xy 133.35 83.82)
 		)
 		(stroke
@@
 	(wire
 		(pts
-			(xy 243.84 60.96) (xy 257.81 60.96)
+			(xy 243.84 60.96) (xy 260.35 60.96)
 		)
 		(stroke
@@
 			)
 		)
-		(property "Footprint" "Resistor_THT:R_Axial_DIN0207_L6.3mm_D2.5mm_P10.16mm_Horizontal"
+		(property "Footprint" "mylib:R_L6.3mm_D2.5mm_P10.16mm_Horizontal_reversible"
 			(at 68.326 118.364 90)
 			(effects
@@
 			)
 		)
-		(property "Footprint" "Capacitor_SMD:C_0805_2012Metric_Pad1.18x1.45mm_HandSolder"
+		(property "Footprint" "mylib:C_0805_2012_HandSolder_reversible"
 			(at 42.8752 138.43 0)
 			(effects
@@
 	)
 	(symbol
+		(lib_id "power:PWR_FLAG")
+		(at 260.35 60.96 0)
+		(unit 1)
+		(exclude_from_sim no)
+		(in_bom yes)
+		(on_board yes)
+		(dnp no)
+		(fields_autoplaced yes)
+		(property "Reference" "#FLG02"
+			(at 260.35 59.055 0)
+			(effects
+				(font
+					(size 1.27 1.27)
+				)
+				(hide yes)
+			)
+		)
+		(property "Value" "PWR_FLAG"
+			(at 260.35 55.88 0)
+			(effects
+				(font
+					(size 1.27 1.27)
+				)
+			)
+		)
+		(property "Footprint" ""
+			(at 260.35 60.96 0)
+			(effects
+				(font
+					(size 1.27 1.27)
+				)
+				(hide yes)
+			)
+		)
+		(property "Datasheet" "~"
+			(at 260.35 60.96 0)
+			(effects
+				(font
+					(size 1.27 1.27)
+				)
+				(hide yes)
+			)
+		)
+		(property "Description" "Special symbol for telling ERC where power comes from"
+			(at 260.35 60.96 0)
+			(effects
+				(font
+					(size 1.27 1.27)
+				)
+				(hide yes)
+			)
+		)
+		(pin "1"
+		)
+		(instances
+			(project "board"
+				(path "/e49ea350-db18-4e55-8e96-c45c407ec11d"
+					(reference "#FLG02")
+					(unit 1)
+				)
+			)
+		)
+	)
+	(symbol
 		(lib_name "KY-023_1")
 		(lib_id "Keyboard:KY-023")
@@
 	)
 	(symbol
-		(lib_id "power:VCC")
-		(at 248.92 64.77 0)
-		(unit 1)
-		(exclude_from_sim no)
-		(in_bom yes)
-		(on_board yes)
-		(dnp no)
-		(fields_autoplaced yes)
-		(property "Reference" "#PWR02"
-			(at 248.92 68.58 0)
-			(effects
-				(font
-					(size 1.27 1.27)
-				)
-				(hide yes)
-			)
-		)
-		(property "Value" "VCC"
-			(at 248.92 59.69 0)
-			(effects
-				(font
-					(size 1.27 1.27)
-				)
-			)
-		)
-		(property "Footprint" ""
-			(at 248.92 64.77 0)
-			(effects
-				(font
-					(size 1.27 1.27)
-				)
-				(hide yes)
-			)
-		)
-		(property "Datasheet" ""
-			(at 248.92 64.77 0)
-			(effects
-				(font
-					(size 1.27 1.27)
-				)
-				(hide yes)
-			)
-		)
-		(property "Description" "Power symbol creates a global label with name \"VCC\""
-			(at 248.92 64.77 0)
-			(effects
-				(font
-					(size 1.27 1.27)
-				)
-				(hide yes)
-			)
-		)
-		(pin "1"
-		)
-		(instances
-			(project ""
-				(path "/e49ea350-db18-4e55-8e96-c45c407ec11d"
-					(reference "#PWR02")
-					(unit 1)
-				)
-			)
-		)
-	)
-	(symbol
 		(lib_id "Switch:SW_Push")
 		(at 52.07 63.5 0)
@@
 	(symbol
 		(lib_id "power:GNDPWR")
-		(at 257.81 60.96 0)
+		(at 260.35 60.96 0)
 		(unit 1)
 		(exclude_from_sim no)
@@
 		(fields_autoplaced yes)
 		(property "Reference" "#PWR01"
-			(at 257.81 66.04 0)
+			(at 260.35 66.04 0)
 			(effects
 				(font
@@
 		)
 		(property "Value" "GNDPWR"
-			(at 257.683 64.77 0)
+			(at 260.223 64.77 0)
 			(effects
 				(font
@@
 		)
 		(property "Footprint" ""
-			(at 257.81 62.23 0)
+			(at 260.35 62.23 0)
 			(effects
 				(font
@@
 		)
 		(property "Datasheet" ""
-			(at 257.81 62.23 0)
+			(at 260.35 62.23 0)
 			(effects
 				(font
@@
 		)
 		(property "Description" "Power symbol creates a global label with name \"GNDPWR\" , global ground"
-			(at 257.81 60.96 0)
+			(at 260.35 60.96 0)
 			(effects
 				(font
@@
 			)
 		)
-		(property "Footprint" "Capacitor_SMD:C_0805_2012Metric_Pad1.18x1.45mm_HandSolder"
+		(property "Footprint" "mylib:C_0805_2012_HandSolder_reversible"
 			(at 68.2752 138.43 0)
 			(effects
@@
 	)
 	(symbol
+		(lib_id "power:VCC")
+		(at 254 57.15 0)
+		(unit 1)
+		(exclude_from_sim no)
+		(in_bom yes)
+		(on_board yes)
+		(dnp no)
+		(fields_autoplaced yes)
+		(property "Reference" "#PWR02"
+			(at 254 60.96 0)
+			(effects
+				(font
+					(size 1.27 1.27)
+				)
+				(hide yes)
+			)
+		)
+		(property "Value" "VCC"
+			(at 254 52.07 0)
+			(effects
+				(font
+					(size 1.27 1.27)
+				)
+			)
+		)
+		(property "Footprint" ""
+			(at 254 57.15 0)
+			(effects
+				(font
+					(size 1.27 1.27)
+				)
+				(hide yes)
+			)
+		)
+		(property "Datasheet" ""
+			(at 254 57.15 0)
+			(effects
+				(font
+					(size 1.27 1.27)
+				)
+				(hide yes)
+			)
+		)
+		(property "Description" "Power symbol creates a global label with name \"VCC\""
+			(at 254 57.15 0)
+			(effects
+				(font
+					(size 1.27 1.27)
+				)
+				(hide yes)
+			)
+		)
+		(pin "1"
+		)
+		(instances
+			(project ""
+				(path "/e49ea350-db18-4e55-8e96-c45c407ec11d"
+					(reference "#PWR02")
+					(unit 1)
+				)
+			)
+		)
+	)
+	(symbol
 		(lib_id "Switch:SW_Push")
 		(at 102.87 50.8 0)
@@
 			)
 		)
-		(property "Footprint" "Resistor_THT:R_Axial_DIN0207_L6.3mm_D2.5mm_P10.16mm_Horizontal"
+		(property "Footprint" "mylib:R_L6.3mm_D2.5mm_P10.16mm_Horizontal_reversible"
 			(at 42.926 118.364 90)
 			(effects
@@
 					(unit 1)
 				)
+			)
+		)
+	)
+	(symbol
+		(lib_id "power:PWR_FLAG")
+		(at 246.38 57.15 0)
+		(unit 1)
+		(exclude_from_sim no)
+		(in_bom yes)
+		(on_board yes)
+		(dnp no)
+		(fields_autoplaced yes)
+		(property "Reference" "#FLG01"
+			(at 246.38 55.245 0)
+			(effects
+				(font
+					(size 1.27 1.27)
+				)
+				(hide yes)
+			)
+		)
+		(property "Value" "PWR_FLAG"
+			(at 246.38 52.07 0)
+			(effects
+				(font
+					(size 1.27 1.27)
+				)
+			)
+		)
+		(property "Footprint" ""
+			(at 246.38 57.15 0)
+			(effects
+				(font
+					(size 1.27 1.27)
+				)
+				(hide yes)
+			)
+		)
+		(property "Datasheet" "~"
+			(at 246.38 57.15 0)
+			(effects
+				(font
+					(size 1.27 1.27)
+				)
+				(hide yes)
+			)
+		)
+		(property "Description" "Special symbol for telling ERC where power comes from"
+			(at 246.38 57.15 0)
+			(effects
+				(font
+					(size 1.27 1.27)
+				)
+				(hide yes)
+			)
+		)
+		(pin "1"
+		)
+		(instances
+			(project ""
+				(path "/e49ea350-db18-4e55-8e96-c45c407ec11d"
+					(reference "#FLG01")
+					(unit 1)
+				)
