File: Kicad/board.kicad_sch (KiCad schematic)
At the start: 45 parts, among them SW1 SW_Push, SW10 SW_Push, SW11 SW_Push, SW12 SW_Push, SW13 RotaryEncoder, SW2 SW_Push, SW3 SW_Push, SW4 SW_Push, SW5 SW_Push, SW6 SW_Push, SW7 SW_Push, SW8 SW_Push, SW9 SW_Push, U1 XIAO-ESP32-S3-DIP, U2 KY-023, U3 OLED, U4 KY-023

Commit message: [!][fix] fix power line connection
Parts:
- U1: footprint XIAO-ESP32S3-DIP:XIAO-ESP32S3-DIP -> mylib:XIAO-ESP32S3_reversible
Connections:
- net OLED_SCL is gone; now on net oled_scl: JP3.2 (B), JP7.2 (B)
- net OLED_SDA is gone; now on net oled_sda: JP4.2 (B), JP8.2 (B)
- net VCC: now also U1.12 (VCC_3V3); no longer U1.14 (VBUS)
Changed lines of the file:
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@@
 	)
 	(junction
-		(at 246.38 57.15)
-		(diameter 0)
-		(color 0 0 0 0)
-	)
-	(junction
 		(at 41.91 124.46)
 		(diameter 0)
@@
 	)
 	(junction
-		(at 260.35 60.96)
-		(diameter 0)
-		(color 0 0 0 0)
-	)
-	(junction
 		(at 57.15 83.82)
 		(diameter 0)
@@
 	)
 	(junction
+		(at 265.43 60.96)
+		(diameter 0)
+		(color 0 0 0 0)
+	)
+	(junction
 		(at 72.39 63.5)
 		(diameter 0)
@@
 	)
 	(no_connect
-		(at 243.84 64.77)
+		(at 137.16 83.82)
 	)
 	(no_connect
-		(at 137.16 83.82)
+		(at 243.84 57.15)
 	)
 	(no_connect
@@
 	(wire
 		(pts
-			(xy 246.38 57.15) (xy 254 57.15)
-		)
-		(stroke
-			(width 0)
-			(type default)
-		)
-	)
-	(wire
-		(pts
 			(xy 107.95 71.12) (xy 133.35 71.12)
 		)
@@
 	(wire
 		(pts
-			(xy 246.38 57.15) (xy 243.84 57.15)
-		)
-		(stroke
-			(width 0)
-			(type default)
-		)
-	)
-	(wire
-		(pts
 			(xy 67.31 121.92) (xy 67.31 129.54)
 		)
@@
 	(wire
 		(pts
-			(xy 243.84 60.96) (xy 260.35 60.96)
+			(xy 243.84 60.96) (xy 265.43 60.96)
 		)
 		(stroke
@@
 	(wire
 		(pts
+			(xy 243.84 64.77) (xy 254 64.77)
+		)
+		(stroke
+			(width 0)
+			(type default)
+		)
+	)
+	(wire
+		(pts
 			(xy 135.89 128.27) (xy 142.24 128.27)
 		)
@@
 		)
 	)
-	(global_label "OLED_SDA"
+	(global_label "oled_sda"
 		(shape input)
 		(at 153.67 134.62 0)
@@
 		)
 		(property "Intersheetrefs" "${INTERSHEET_REFS}"
-			(at 165.9685 134.62 0)
+			(at 165.0007 134.62 0)
 			(effects
 				(font
@@
 		)
 	)
-	(global_label "OLED_SCL"
+	(global_label "oled_scl"
 		(shape input)
 		(at 153.67 128.27 0)
@@
 		)
 		(property "Intersheetrefs" "${INTERSHEET_REFS}"
-			(at 165.908 128.27 0)
+			(at 164.4565 128.27 0)
 			(effects
 				(font
@@
 		)
 	)
-	(global_label "OLED_SDA"
+	(global_label "oled_sda"
 		(shape input)
 		(at 153.67 158.75 0)
@@
 		)
 		(property "Intersheetrefs" "${INTERSHEET_REFS}"
-			(at 165.9685 158.75 0)
+			(at 165.0007 158.75 0)
 			(effects
 				(font
@@
 		)
 	)
-	(global_label "OLED_SCL"
+	(global_label "oled_scl"
 		(shape input)
 		(at 153.67 152.4 0)
@@
 		)
 		(property "Intersheetrefs" "${INTERSHEET_REFS}"
-			(at 165.908 152.4 0)
+			(at 164.4565 152.4 0)
 			(effects
 				(font
@@
 	(symbol
 		(lib_id "power:PWR_FLAG")
-		(at 260.35 60.96 0)
+		(at 265.43 60.96 0)
 		(unit 1)
 		(exclude_from_sim no)
@@
 		(fields_autoplaced yes)
 		(property "Reference" "#FLG02"
-			(at 260.35 59.055 0)
+			(at 265.43 59.055 0)
 			(effects
 				(font
@@
 		)
 		(property "Value" "PWR_FLAG"
-			(at 260.35 55.88 0)
+			(at 265.43 55.88 0)
 			(effects
 				(font
@@
 		)
 		(property "Footprint" ""
-			(at 260.35 60.96 0)
+			(at 265.43 60.96 0)
 			(effects
 				(font
@@
 		)
 		(property "Datasheet" "~"
-			(at 260.35 60.96 0)
+			(at 265.43 60.96 0)
 			(effects
 				(font
@@
 		)
 		(property "Description" "Special symbol for telling ERC where power comes from"
-			(at 260.35 60.96 0)
+			(at 265.43 60.96 0)
 			(effects
 				(font
@@
 	(symbol
 		(lib_id "power:GNDPWR")
-		(at 260.35 60.96 0)
+		(at 265.43 60.96 0)
 		(unit 1)
 		(exclude_from_sim no)
@@
 		(fields_autoplaced yes)
 		(property "Reference" "#PWR01"
-			(at 260.35 66.04 0)
+			(at 265.43 66.04 0)
 			(effects
 				(font
@@
 		)
 		(property "Value" "GNDPWR"
-			(at 260.223 64.77 0)
+			(at 265.303 64.77 0)
 			(effects
 				(font
@@
 		)
 		(property "Footprint" ""
-			(at 260.35 62.23 0)
+			(at 265.43 62.23 0)
 			(effects
 				(font
@@
 		)
 		(property "Datasheet" ""
-			(at 260.35 62.23 0)
+			(at 265.43 62.23 0)
 			(effects
 				(font
@@
 		)
 		(property "Description" "Power symbol creates a global label with name \"GNDPWR\" , global ground"
-			(at 260.35 60.96 0)
+			(at 265.43 60.96 0)
 			(effects
 				(font
@@
 	(symbol
 		(lib_id "power:VCC")
-		(at 254 57.15 0)
+		(at 254 64.77 0)
 		(unit 1)
 		(exclude_from_sim no)
@@
 		(fields_autoplaced yes)
 		(property "Reference" "#PWR02"
-			(at 254 60.96 0)
+			(at 254 68.58 0)
 			(effects
 				(font
@@
 		)
 		(property "Value" "VCC"
-			(at 254 52.07 0)
+			(at 254 59.69 0)
 			(effects
 				(font
@@
 		)
 		(property "Footprint" ""
-			(at 254 57.15 0)
+			(at 254 64.77 0)
 			(effects
 				(font
@@
 		)
 		(property "Datasheet" ""
-			(at 254 57.15 0)
+			(at 254 64.77 0)
 			(effects
 				(font
@@
 		)
 		(property "Description" "Power symbol creates a global label with name \"VCC\""
-			(at 254 57.15 0)
+			(at 254 64.77 0)
 			(effects
 				(font
@@
 		)
 		(instances
-			(project ""
+			(project "board"
 				(path "/e49ea350-db18-4e55-8e96-c45c407ec11d"
 					(reference "#PWR02")
@@
 	)
 	(symbol
-		(lib_id "power:PWR_FLAG")
-		(at 246.38 57.15 0)
-		(unit 1)
-		(exclude_from_sim no)
-		(in_bom yes)
-		(on_board yes)
-		(dnp no)
-		(fields_autoplaced yes)
-		(property "Reference" "#FLG01"
-			(at 246.38 55.245 0)
-			(effects
-				(font
-					(size 1.27 1.27)
-				)
-				(hide yes)
-			)
-		)
-		(property "Value" "PWR_FLAG"
-			(at 246.38 52.07 0)
-			(effects
-				(font
-					(size 1.27 1.27)
-				)
-			)
-		)
-		(property "Footprint" ""
-			(at 246.38 57.15 0)
-			(effects
-				(font
-					(size 1.27 1.27)
-				)
-				(hide yes)
-			)
-		)
-		(property "Datasheet" "~"
-			(at 246.38 57.15 0)
-			(effects
-				(font
-					(size 1.27 1.27)
-				)
-				(hide yes)
-			)
-		)
-		(property "Description" "Special symbol for telling ERC where power comes from"
-			(at 246.38 57.15 0)
-			(effects
-				(font
-					(size 1.27 1.27)
-				)
-				(hide yes)
-			)
-		)
-		(pin "1"
-		)
-		(instances
-			(project ""
-				(path "/e49ea350-db18-4e55-8e96-c45c407ec11d"
-					(reference "#FLG01")
-					(unit 1)
-				)
-			)
-		)
-	)
-	(symbol
 		(lib_id "Jumper:SolderJumper_2_Open")
 		(at 146.05 152.4 0)
@@
 			)
 		)
-		(property "Footprint" "XIAO-ESP32S3-DIP:XIAO-ESP32S3-DIP"
+		(property "Footprint" "mylib:XIAO-ESP32S3_reversible"
 			(at 216.408 83.82 0)
 			(effects
